Commit message: fixed vmecanumrover.xacro

File: urdf/vmecanumrover.xacro (robot description, xacro)
@@ -380,18 +380,18 @@
   <!-- back -->
   <xacro:bumperbaseboard prefix="back" parent="body_link" xyz="-0.196 0 0.0365" z_dir="-90"/>
-  <!-- base attachment(LiDER,emergency button,wyreless charge) board(front) -->
+  <!-- base attachment(LiDAR,emergency button,wyreless charge) board(front) -->
   <!--  upper side  -->
 <!--  <xacro:optionattachboard prefix="front" xyz="0.157 0 0.1665" z_dir="0" /> -->
   <!--  lower side  -->
   <xacro:optionattachboard prefix="front" xyz="0.157 0 0.1585" z_dir="0" />
-  <!-- base attachment(LiDER,emergency button,wyreless charge) board(back) -->
+  <!-- base attachment(LiDAR,emergency button,wyreless charge) board(back) -->
   <!--  upper side  -->
 <!--  <xacro:optionattachboard prefix="back" xyz="-0.157 0 0.1665" z_dir="180" /> -->
   <!--  lower side  -->
   <xacro:optionattachboard prefix="back" xyz="-0.157 0 0.1585" z_dir="180" />
-  <!-- LiDER  -->
-  <joint name="lider_joint" type="fixed">
+  <!-- LiDAR  -->
+  <joint name="lidar_joint" type="fixed">
     <parent link="board_front_link"/>
-    <child  link="lider_link"/>
+    <child  link="laser"/>
   <!-- attach upper side -->
 <!--    <origin xyz="0.042 0 0.0570" rpy="0 0 0"/> -->
@@ -399,8 +399,8 @@
     <origin xyz="0.042 0 -0.0570" rpy="${radians(180)} 0 0"/>
   </joint>
-  <link name="lider_link">
-    <visual>
-      <geometry>
-          <mesh filename="package://mecanumrover_samples/meshes/dae/mecanum_lider.dae" />
+  <link name="laser">
+    <visual>
+      <geometry>
+          <mesh filename="package://mecanumrover_samples/meshes/dae/mecanum_lidar.dae" />
       </geometry>
       <material name="black"/>
@@ -408,5 +408,5 @@
     <collision>
       <geometry>
-          <mesh filename="package://mecanumrover_samples/meshes/stl/mecanum_lider.stl" />
+          <mesh filename="package://mecanumrover_samples/meshes/stl/mecanum_lidar.stl" />
       </geometry>
     </collision>
@@ -415,5 +415,5 @@
     </inertial>
   </link>
-  <gazebo reference="lider_link">
+  <gazebo reference="laser">
     <material>Gazebo/Black</material>
     <sensor type="ray" name="lrf_sensor">
